File: PU22_ram_mod.kicad_pcb (KiCad board)
At the start: 2 copper layers, 39.2 x 94.7 mm, 11 parts, among them J1 MOBO, J2 BA8, J3 BA10

Commit message: Some tracing
Routing:
- net GND: track 94.8 -> 37.1 mm
- net /A7: track 2.78 -> 47.4 mm
- net /A9: track 4.32 -> 46.5 mm
- net /~{OE}: track 7.91 -> 48.3 mm
- net VCC: track 71.8 -> 35.2 mm, vias 2 -> 0
- net /D12: track 0.00 -> 16.2 mm
- net /D13: track 0.00 -> 15.6 mm
- net /D14: track 0.00 -> 14.7 mm
- net /D15: track 0.00 -> 13.8 mm
- net unconnected-(J1-Pin_40-Pad40): track 5.20 -> 0.00 mm
- net /A11: track 3.67 -> 0.00 mm
- net /D30: track 31.9 -> 28.9 mm, vias 0 -> 1
- net /D29: track 31.0 -> 28.0 mm, vias 0 -> 1
- net /D31: track 32.4 -> 29.7 mm, vias 0 -> 1
- net /D28: track 29.8 -> 27.1 mm, vias 0 -> 1
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Other:
- board size 39.2 x 94.7 mm -> 57.3 x 93.7 mm

Commit message: some more organizing
Routing:
- net /A7: track 47.4 -> 3.04 mm
- net /A9: track 46.5 -> 4.72 mm
- net /~{OE}: track 48.3 -> 8.00 mm
- net VCC: track 35.2 -> 63.5 mm
- net GND: track 37.1 -> 64.6 mm
Other:
- board size 57.3 x 93.7 mm -> 39.2 x 94.7 mm
Changed lines of the file:
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@@
 	)
 	(gr_arc
-		(start 98.934 50.292)
-		(mid 99.08279 49.93279)
-		(end 99.442 49.784)
+		(start 116.968 49.276)
+		(mid 117.11679 48.91679)
+		(end 117.476 48.768)
 		(stroke
 			(width 0.05)
@@
 	)
 	(gr_line
-		(start 108.204 50.292)
-		(end 108.204 87.73521)
+		(start 126.238 49.276)
+		(end 126.238 86.71921)
 		(stroke
 			(width 0.05)
@@
 	)
 	(gr_line
-		(start 99.442 49.784)
-		(end 107.696 49.784)
+		(start 117.476 48.768)
+		(end 125.73 48.768)
 		(stroke
 			(width 0.05)
@@
 	)
 	(gr_line
-		(start 98.934 50.292)
-		(end 98.934 84.074)
+		(start 116.968 49.276)
+		(end 116.968 83.058)
 		(stroke
 			(width 0.05)
@@
 	)
 	(gr_arc
-		(start 107.696 49.784)
-		(mid 108.05521 49.93279)
-		(end 108.204 50.292)
+		(start 125.73 48.768)
+		(mid 126.08921 48.91679)
+		(end 126.238 49.276)
 		(stroke
 			(width 0.05)
@@
 	)
 	(segment
+		(start 152.019 96.901)
+		(end 152.738 97.62)
+		(width 0.2)
+		(layer "B.Cu")
+		(net 1)
+	)
+	(segment
+		(start 148.5855 96.901)
+		(end 152.019 96.901)
+		(width 0.2)
+		(layer "B.Cu")
+		(net 1)
+	)
+	(segment
+		(start 135.466 141.14)
+		(end 135.466 138.43)
+		(width 0.2)
+		(layer "B.Cu")
+		(net 1)
+	)
+	(segment
+		(start 134.747 96.901)
+		(end 131.3135 96.901)
+		(width 0.2)
+		(layer "B.Cu")
+		(net 1)
+	)
+	(segment
+		(start 134.747 141.859)
+		(end 135.466 141.14)
+		(width 0.2)
+		(layer "B.Cu")
+		(net 1)
+	)
+	(segment
+		(start 152.738 97.62)
+		(end 152.738 100.203)
+		(width 0.2)
+		(layer "B.Cu")
+		(net 1)
+	)
+	(segment
+		(start 148.5855 141.859)
+		(end 152.019 141.859)
+		(width 0.2)
+		(layer "B.Cu")
+		(net 1)
+	)
+	(segment
+		(start 152.019 141.859)
+		(end 152.738 141.14)
+		(width 0.2)
+		(layer "B.Cu")
+		(net 1)
+	)
+	(segment
+		(start 135.466 97.62)
+		(end 134.747 96.901)
+		(width 0.2)
+		(layer "B.Cu")
+		(net 1)
+	)
+	(segment
+		(start 131.3135 141.859)
+		(end 134.747 141.859)
+		(width 0.2)
+		(layer "B.Cu")
+		(net 1)
+	)
+	(segment
+		(start 135.466 100.203)
+		(end 135.466 97.62)
+		(width 0.2)
+		(layer "B.Cu")
+		(net 1)
+	)
+	(segment
+		(start 152.738 141.14)
+		(end 152.738 138.43)
+		(width 0.2)
+		(layer "B.Cu")
+		(net 1)
+	)
+	(segment
 		(start 125.338001 49.34)
 		(end 125.038 49.640001)
@@
 		(width 0.2)
 		(layer "F.Cu")
+		(net 2)
+	)
+	(segment
+		(start 141.478 97.536)
+		(end 141.478 100.203)
+		(width 0.2)
+		(layer "B.Cu")
+		(net 2)
+	)
+	(segment
+		(start 142.367 141.859)
+		(end 141.478 140.97)
+		(width 0.2)
+		(layer "B.Cu")
+		(net 2)
+	)
+	(segment
+		(start 142.113 96.901)
+		(end 141.478 97.536)
+		(width 0.2)
+		(layer "B.Cu")
+		(net 2)
+	)
+	(segment
+		(start 128.1885 96.901)
+		(end 124.841 96.901)
+		(width 0.2)
+		(layer "B.Cu")
+		(net 2)
+	)
+	(segment
+		(start 124.206 97.536)
+		(end 124.206 100.203)
+		(width 0.2)
+		(layer "B.Cu")
+		(net 2)
+	)
+	(segment
+		(start 124.841 96.901)
+		(end 124.206 97.536)
+		(width 0.2)
+		(layer "B.Cu")
+		(net 2)
+	)
+	(segment
+		(start 145.4605 96.901)
+		(end 142.113 96.901)
+		(width 0.2)
+		(layer "B.Cu")
+		(net 2)
+	)
+	(segment
+		(start 125.349 141.859)
+		(end 124.206 140.716)
+		(width 0.2)
+		(layer "B.Cu")
+		(net 2)
+	)
+	(segment
+		(start 124.206 140.716)
+		(end 124.206 138.43)
+		(width 0.2)
+		(layer "B.Cu")
+		(net 2)
+	)
+	(segment
+		(start 141.478 140.97)
+		(end 141.478 138.43)
+		(width 0.2)
+		(layer "B.Cu")
+		(net 2)
+	)
+	(segment
+		(start 128.1885 141.859)
+		(end 125.349 141.859)
+		(width 0.2)
+		(layer "B.Cu")
+		(net 2)
+	)
+	(segment
+		(start 145.4605 141.859)
+		(end 142.367 141.859)
+		(width 0.2)
+		(layer "B.Cu")
 		(net 2)
 	)
@@
 	)
 	(segment
-		(start 124.768 89.744843)
-		(end 125.193157 90.17)
+		(start 126.238 74.14)
+		(end 125.338001 74.14)
 		(width 0.1)
 		(layer "B.Cu")
@@
 	)
 	(segment
-		(start 129.794 90.17)
-		(end 130.102 90.478)
-		(width 0.1)
-		(layer "B.Cu")
-		(net 26)
-	)
-	(segment
-		(start 130.102 108.404)
-		(end 129.413 109.093)
+		(start 124.768 76.192843)
+		(end 124.768 77.724)
 		(width 0.1)
 		(layer "B.Cu")
@@
 	)
 	(segment
-		(start 129.413 109.093)
-		(end 124.206 109.093)
-		(width 0.1)
-		(layer "B.Cu")
-		(net 26)
-	)
-	(segment
 		(start 124.768 74.710001)
-		(end 124.768 89.744843)
-		(width 0.1)
-		(layer "B.Cu")
-		(net 26)
-	)
-	(segment
-		(start 125.193157 90.17)
-		(end 129.794 90.17)
-		(width 0.1)
-		(layer "B.Cu")
-		(net 26)
-	)
-	(segment
-		(start 130.102 90.478)
-		(end 130.102 108.404)
-		(width 0.1)
-		(layer "B.Cu")
-		(net 26)
-	)
-	(segment
-		(start 126.238 74.14)
-		(end 125.338001 74.14)
+		(end 124.768 76.192843)
 		(width 0.1)
 		(layer "B.Cu")
@@
 	)
 	(segment
-		(start 129.902 107.334)
-		(end 129.902 90.786)
+		(start 125.338001 70.94)
+		(end 124.568 71.710001)
 		(width 0.1)
 		(layer "B.Cu")
@@
 	)
 	(segment
-		(start 124.206 107.823)
-		(end 129.413 107.823)
+		(start 124.568 74.792843)
+		(end 124.568 77.724)
 		(width 0.1)
 		(layer "B.Cu")
@@
 	)
 	(segment
-		(start 129.54 90.424)
-		(end 125.164315 90.424)
+		(start 124.568 71.710001)
+		(end 124.568 74.792843)
 		(width 0.1)
 		(layer "B.Cu")
@@
 	)
 	(segment
-		(start 125.338001 70.94)
-		(end 126.238 70.94)
+		(start 126.238 70.94)
+		(end 125.338001 70.94)
 		(width 0.1)
 		(layer "B.Cu")
@@
 	)
 	(segment
-		(start 124.568 89.827685)
-		(end 124.568 71.710001)
-		(width 0.1)
-		(layer "B.Cu")
-		(net 57)
-	)
-	(segment
-		(start 129.413 107.823)
-		(end 129.902 107.334)
-		(width 0.1)
-		(layer "B.Cu")
-		(net 57)
-	)
-	(segment
-		(start 125.164315 90.424)
-		(end 124.568 89.827685)
-		(width 0.1)
-		(layer "B.Cu")
-		(net 57)
-	)
-	(segment
-		(start 124.568 71.710001)
-		(end 125.338001 70.94)
-		(width 0.1)
-		(layer "B.Cu")
-		(net 57)
-	)
-	(segment
-		(start 129.902 90.786)
-		(end 129.54 90.424)
-		(width 0.1)
-		(layer "B.Cu")
-		(net 57)
-	)
-	(segment
-		(start 130.048 89.916)
-		(end 125.222 89.916)
+		(start 126.238 75.74)
+		(end 125.338001 75.74)
 		(width 0.1)
 		(layer "B.Cu")
@@
 	)
 	(segment
-		(start 125.222 89.916)
-		(end 124.968 89.662)
+		(start 124.968 76.110001)
+		(end 124.968 77.724)
 		(width 0.1)
 		(layer "B.Cu")
@@
 	)
 	(segment
-		(start 130.302 110.49)
-		(end 130.302 90.17)
-		(width 0.1)
-		(layer "B.Cu")
-		(net 58)
-	)
-	(segment
-		(start 124.968 89.662)
+		(start 125.338001 75.74)
 		(end 124.968 76.110001)
 		(width 0.1)
 		(layer "B.Cu")
-		(net 58)
-	)
-	(segment
-		(start 124.206 111.633)
-		(end 129.159 111.633)
-		(width 0.1)
-		(layer "B.Cu")
-		(net 58)
-	)
-	(segment
-		(start 124.968 76.110001)
-		(end 125.338001 75.74)
-		(width 0.1)
-		(layer "B.Cu")
-		(net 58)
-	)
-	(segment
-		(start 125.338001 75.74)
-		(end 126.238 75.74)
-		(width 0.1)
-		(layer "B.Cu")
-		(net 58)
-	)
-	(segment
-		(start 129.159 111.633)
-		(end 130.302 110.49)
-		(width 0.1)
-		(layer "B.Cu")
-		(net 58)
-	)
-	(segment
-		(start 130.302 90.17)
-		(end 130.048 89.916)
-		(width 0.1)
-		(layer "B.Cu")

Commit message: Some tracing
Parts:
- moved J2 3.81 mm to (153.7, 90.7)
- moved J3 3.81 mm to (149.9, 90.7)
Routing:
- net /A8: track 0.00 -> 136.1 mm, vias 0 -> 2
- net /A10: track 0.00 -> 119.6 mm, vias 0 -> 4
- net /A7: track 3.04 -> 80.9 mm, vias 0 -> 2
- net /~{RAS}: track 8.93 -> 79.8 mm, vias 0 -> 2
- net /~{OE}: track 8.00 -> 76.8 mm, vias 0 -> 2
- net /A9: track 4.72 -> 72.3 mm, vias 0 -> 2
- net /A0: track 8.29 -> 74.8 mm, vias 0 -> 2
- net /A1: track 7.19 -> 72.2 mm, vias 0 -> 2
- net /A6: track 2.99 -> 67.4 mm, vias 0 -> 2
- net /A5: track 3.89 -> 67.1 mm, vias 0 -> 2
- net /A2: track 6.54 -> 69.5 mm, vias 0 -> 2
- net /A4: track 4.77 -> 65.9 mm
- net /A3: track 5.66 -> 66.7 mm, vias 0 -> 2
- net /~{WE}: track 8.89 -> 44.5 mm

Commit message: Some routing
Connections:
- U3 pad 2: /D17 -> /D16
- U3 pad 24: /D21 -> /D20
- U3 pad 25: /D22 -> /D21
- U3 pad 26: /D23 -> /D22
- U3 pad 27: /D24 -> /D23
- U3 pad 3: /D18 -> /D17
- U3 pad 4: /D19 -> /D18
- U3 pad 5: /D20 -> /D19
- U4 pad 2: /D25 -> /D24
- U4 pad 24: /D29 -> /D28
- U4 pad 25: /D30 -> /D29
- U4 pad 26: /D31 -> /D30
- U4 pad 27: /D32 -> /D31
- U4 pad 3: /D26 -> /D25
- U4 pad 4: /D27 -> /D26
- U4 pad 5: /D28 -> /D27
Routing:
- net /D20: track 17.9 -> 97.3 mm, vias 0 -> 2
- net /D22: track 19.7 -> 95.1 mm, vias 0 -> 2
- net /D19: track 16.2 -> 91.1 mm, vias 0 -> 2
- net /D18: track 15.6 -> 89.1 mm, vias 0 -> 2
- net /D23: track 20.6 -> 93.3 mm, vias 0 -> 2
- net /D17: track 14.7 -> 87.2 mm, vias 0 -> 2
- net /D16: track 13.8 -> 85.8 mm, vias 0 -> 2
- net /D21: track 18.8 -> 85.7 mm, vias 0 -> 2
- net /~{CAS3}: track 10.6 -> 75.6 mm, vias 0 -> 2
- net /D24: track 23.2 -> 84.6 mm, vias 0 -> 2
- net /~{CAS4}: track 9.77 -> 67.6 mm, vias 0 -> 2
- net /A9: track 72.3 -> 126.7 mm, vias 2 -> 4
- net /A3: track 66.7 -> 119.1 mm, vias 2 -> 7
- net /~{OE}: track 76.8 -> 127.9 mm, vias 2 -> 4
- net /A2: track 69.5 -> 119.7 mm, vias 2 -> 7
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
Commit message: Routing
Routing:
- net VCC: track 63.5 -> 311.1 mm, vias 0 -> 7
- net GND: track 64.6 -> 223.9 mm, vias 0 -> 12
- net /D25: track 24.4 -> 96.8 mm, vias 1 -> 4
- net /D27: track 26.1 -> 98.2 mm, vias 1 -> 4
- net /D26: track 25.5 -> 97.5 mm, vias 1 -> 4
- net /D3: track 27.3 -> 94.5 mm, vias 1 -> 4
- net /D28: track 27.1 -> 93.0 mm, vias 1 -> 4
- net /D29: track 28.0 -> 92.0 mm, vias 1 -> 4
- net /D2: track 28.5 -> 91.9 mm, vias 1 -> 2
- net /D1: track 29.3 -> 92.0 mm, vias 1 -> 4
- net /D30: track 28.9 -> 91.3 mm, vias 1 -> 4
- net /D0: track 29.9 -> 91.2 mm, vias 1 -> 2
- net /D31: track 29.7 -> 90.0 mm, vias 1 -> 4
- net /D4: track 26.1 -> 76.7 mm, vias 1 -> 2
- net /D5: track 25.1 -> 75.0 mm, vias 1 -> 2
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